File: schematics/patchbay8in8out/patchbay8in8out/patchbay8in8out.sch (KiCad schematic (older format))
At the start: 10 parts

Commit message: schematic progress
Parts:
- added J? (x2): Conn_01x08_Male, symbol Connector:Conn_01x08_Male
- added J?: Conn_01x09_Male, symbol Connector:Conn_01x09_Male
Connections:
- net at U?.1 (QB): now also R?.2
- net VCC: now reaches U?.10 (~SRCLR)
- net VCC: now also U?.16 (VCC), J?.1 (Pin_1)
- net at U?.11 (SRCLK): now also J?.3 (Pin_3)
- net at U?.12 (RCLK): now also J?.4 (Pin_4)
- net GND: now reaches U?.13 (~OE)
- net GND: now also U?.8 (GND), U?.8 (GND), J?.9 (Pin_9)
- net at U?.14 (SER): now also J?.2 (Pin_2)
- net at U?.15 (QA): now also R?.2
- net at U?.2 (QC): now also R?.2
- net at U?.3 (QD): now also R?.2
- net at U?.4 (QE): now also R?.2
- net at U?.5 (QF): now also R?.2
- net at U?.6 (QG): now also R?.2
- net at U?.7 (QH): now also R?.2
- net at U?.1 (~PL): now also J?.5 (Pin_5)
- net at U?.11 (D0): now also J?.1 (Pin_1)
- net at U?.12 (D1): now also J?.2 (Pin_2)
- net at U?.13 (D2): now also J?.3 (Pin_3)
- net at U?.14 (D3): now also J?.4 (Pin_4)
- net at U?.15 (~CE): now also J?.7 (Pin_7)
- net at U?.2 (CP): now also J?.6 (Pin_6)
- net at U?.3 (D4): now also J?.5 (Pin_5)
- net at U?.4 (D5): now also J?.6 (Pin_6)
- net at U?.5 (D6): now also J?.7 (Pin_7)
- net at U?.6 (D7): now also J?.8 (Pin_8)
- net at U?.9 (Q7): now also J?.8 (Pin_8)
- net at R?.1: now also J?.1 (Pin_1)
- net at R?.1: now also J?.2 (Pin_2)
- net at R?.1: now also J?.3 (Pin_3)
- net at R?.1: now also J?.4 (Pin_4)
- net at R?.1: now also J?.5 (Pin_5)
- net at R?.1: now also J?.6 (Pin_6)
- net at R?.1: now also J?.7 (Pin_7)
- net at R?.1: now also J?.8 (Pin_8)
- no-connect marks 0 -> 3
Other:
- note added: "maybe diodes instead?"
- note added: "oops forgot need pull-down resistors"
- moved on the sheet: U?
