File: schematics/polymod_proto_1/polymod_proto_1/polymod_proto_1.kicad_sch (KiCad schematic)
At the start: 12 parts

Commit message: playing around with electrosmith daisy boards, bit of a mess right now
Parts:
- added ?: ES_DAISY_PATCH_SM_REV1, symbol ES_Daisy_Patch_SM_FB_Rev1-eagle-import:ES_DAISY_PATCH_SM_REV1
- added A?: Device_Audio_Electrosmith_Daisy_Seed_Rev4, daisy-seed:Device_Audio_Electrosmith_Daisy_Seed, symbol Device_Audio_Electrosmith_Daisy_Seed:Device_Audio_Electrosmith_Daisy_Seed_Rev4
Connections:
- net 4051_1: now also A?.22 (ADC_INP10)
- net 4051_2: now also A?.23 (ADC_INP15)
- net 4051_3: now also A?.24 (ADC_INP5)
- net MIDI_IN: now also A?.15 (USART1_RX)
- net MIDI_OUT: now also A?.14 (USART1_TX)
- net PATCHING_IN_CE: now also A?.4 (SDMMC1_D1)
- net PATCHING_IN_CLOCK: now also A?.3 (SDMMC1_D2)
- net PATCHING_IN_DATA: now also A?.5 (SDMMC1_D0)
- net PATCHING_IN_LOAD: now also A?.2 (SDMMC1_D3)
- net PATCHING_OUT_CLOCK: now also A?.27 (ADC_INP11)
- net PATCHING_OUT_DATA: now also A?.26 (ADC_INP3)
- net PATCHING_OUT_LATCH: now also A?.28 (ADC1_INP4)
- net UTILITY_CLOCK: now also A?.29 (DAC1_OUT2)
- net UTILITY_DATA: now also A?.25 (ADC_INP7)
- net UTILITY_LATCH: now also A?.30 (DAC1_OUT1)
- new net: ?.A4 (GND), ?.A7 (GND)

Commit message: schematic is getting somewhere
Parts:
- removed A?: Device_Audio_Electrosmith_Daisy_Seed_Rev4, daisy-seed:Device_Audio_Electrosmith_Daisy_Seed, symbol Device_Audio_Electrosmith_Daisy_Seed:Device_Audio_Electrosmith_Daisy_Seed_Rev4
- removed U?: Teensy4.1, symbol teensy:Teensy4.1
- added D? (x5): LED, symbol Device:LED
- added H? (x4): MountingHole, symbol Mechanical:MountingHole
- added J? (x2): AudioJack2, symbol Connector:AudioJack2
- added J?: Barrel_Jack, symbol Connector:Barrel_Jack
- added R? (x5): 680R, symbol Device:R
- added SW? (x8): SW_Push, symbol Switch:SW_Push
- added U?: 74HC595, symbol 74xx:74HC595
- added U?: 74LS165, symbol 74xx:74LS165
Connections:
- net 4051_1: now also ?.A2 (UART_RX)
- net 4051_2: now also ?.A3 (UART_TX)
- net 4051_ADDRESS_A: now also U?.15 (QA)
- net 4051_ADDRESS_B: now also U?.1 (QB)
- net 4051_ADDRESS_C: now also U?.2 (QC)
- net GND: now also D?.1 (K), D?.1 (K), D?.1 (K), D?.1 (K), D?.1 (K), SW?.1, SW?.1, SW?.1, SW?.1, SW?.1, SW?.1, SW?.1, SW?.1, U?.13 (~{OE}), U?.8 (GND), U?.8 (GND)
- net MIDI_IN: now also ?.A9 (USB_DP)
- net MIDI_OUT: now also ?.A8 (USB_DM)
- net PATCHING_IN_CE: now also ?.D5 (SDMMC_D0), U?.15 (~{CE})
- net PATCHING_IN_CLOCK: now also ?.D7 (SDMMC_CMD), U?.2 (CP)
- net PATCHING_IN_DATA: now also ?.D4 (SDMMC_D1)
- net PATCHING_IN_LOAD: now also ?.D6 (SDMMC_CK), U?.1 (~{PL})
- net PATCHING_OUT_CLOCK: now also ?.D3 (SDMMC_D2), U?.11 (SRCLK)
- net PATCHING_OUT_DATA: now also ?.D1 (SPI_NSS)
- net PATCHING_OUT_LATCH: now also ?.D2 (SDMMC_D3), U?.12 (RCLK)
- net VCC: now also U?.10 (~{SRCLR}), U?.16 (VCC), U?.16 (VCC)
- new net: R?.1, U?.3 (QD)
- new net: R?.1, U?.4 (QE)
- new net: R?.1, U?.5 (QF)
- new net: R?.1, U?.6 (QG)
- new net: R?.1, U?.7 (QH)
- new net: SW?.2, U?.14 (D3)
- new net: SW?.2, U?.11 (D0)
- new net: D?.2 (A), R?.2 (x5)
- new net: SW?.2, U?.5 (D6)
- new net: SW?.2, U?.4 (D5)
- new net: SW?.2, U?.6 (D7)
- new net: SW?.2, U?.12 (D1)
- new net: SW?.2, U?.13 (D2)
- new net: SW?.2, U?.3 (D4)
- new net INPUT: U?.10 (DS)
- new net OUTPUT: U?.9 (Q7)
- no-connect marks 33 -> 9
Other:
- removed sheet Input group 5
- removed sheet Input group 6
- removed sheet Input group 7
- removed sheet Input group 8
- removed sheet Output group 5
- removed sheet Output group 6
- removed sheet Output group 7
- removed sheet Output group 8
- removed sheet Pot group 3
- removed sheet Pot group 4
- note added: "ALTERNATIVELY actually use Daisy Seed for this project but retaining limited pin usage so can use Patch in future"
- note added: "First four 165s handle patching inputs (32 inputs). Subsequent ones handle other digital input, e.g. buttons, switches."
- note added: "First four 595s handle patching outputs (32 outputs). Subsequent ones handle other digital output, e.g. addressing 4051s and controlling LEDs."
- note added: "Need to add four headers to connect Daisy Patch to PCB"
- note added: "Replace DIN with TRS and probably also get rid of MIDI output"

Commit message: schematic nearly done
Parts:
- removed ?: ES_DAISY_PATCH_SM_REV1, symbol ES_Daisy_Patch_SM_FB_Rev1-eagle-import:ES_DAISY_PATCH_SM_REV1
- removed J? (x2): DIN-5_180degree, drumkidcustom:MIDI_DIN5, symbol Connector:DIN-5_180degree
- removed SW?: SW_SPDT, drumkidcustom:EG1206, symbol Switch:SW_SPDT
- added A?: Device_Audio_Electrosmith_Daisy_Seed_Rev4, daisy-seed:Device_Audio_Electrosmith_Daisy_Seed, symbol Device_Audio_Electrosmith_Daisy_Seed:Device_Audio_Electrosmith_Daisy_Seed_Rev4
- added J? (x2): AudioJack3, symbol Connector:AudioJack3
- added JP?: Jumper_2_Open, symbol Jumper:Jumper_2_Open
Connections:
- net 4051_1: now also A?.22 (ADC_INP10)
- net 4051_2: now also A?.23 (ADC_INP15)
- net GND: now also J?.1, A?.40 (GND), J?.S
- net MIDI_IN: now also A?.15 (USART1_RX), JP?.2 (B)
- net MIDI_OUT: now also A?.14 (USART1_TX)
- net PATCHING_IN_CE: now also A?.5 (SDMMC1_D0)
- net PATCHING_IN_CLOCK: now also A?.6 (SDMMC1_CMD)
- net PATCHING_IN_DATA: now also A?.4 (SDMMC1_D1)
- net PATCHING_IN_LOAD: now also A?.7 (SDMMC1_CK)
- net PATCHING_OUT_CLOCK: now also A?.3 (SDMMC1_D2)
- net PATCHING_OUT_DATA: now also A?.8 (SPI1_NSS)
- net PATCHING_OUT_LATCH: now also A?.2 (SDMMC1_D3)
- net VCC: now also R?.1; no longer R?.2
- net UTIL_595: now reaches U?.14 (SER)
- net at R?.2: now also J?.R
- net at D?.2 (A), U?.3 (C2): now also J?.T
- net at R?.2, U?.6 (VO2): now also JP?.1 (A)
- net GNDA: now reaches J?.S
- net GNDA: now also J?.S, A?.20 (AGND)
- net at J?.T: now also A?.18 (AUDIO_OUT_L)
- net at J?.2: now also A?.39 (VIN)
- net at J?.T: now also A?.16 (AUDIO_IN_L)
- net at R?.1: now also J?.T
- net INPUT: no longer names the net of U?.10 (DS)
- net OUTPUT renamed UTIL_165
- new net: J?.R, R?.2
- no-connect marks 9 -> 28
Other:
- note added: "MIDI input socket (TRS type A)"
- note added: "MIDI output socket (TRS type A)"
- note added: "Power input 5.5mm x 2.1mm Centre negative"
- note added: "shield"
- note added: "sink"
- note added: "source"
- note removed: "ALTERNATIVELY actually use Daisy Seed for this project but retaining limited pin usage so can use Patch in future"
- note removed: "MIDI IN"
- note removed: "MIDI OUT"
- note removed: "Need to add four headers to connect Daisy Patch to PCB"
- note removed: "Replace DIN with TRS and probably also get rid of MIDI output"
- moved on the sheet: C?, D?, H?, J?, R?, SW?, U?

Commit message: pcb layout about to start
Parts:
- removed C?: 470uF, Capacitor_THT:CP_Radial_D6.3mm_P2.50mm, symbol Device:CP
- removed J? (x2): AudioJack3, symbol Connector:AudioJack3
- removed J? (x2): AudioJack2, symbol Connector:AudioJack2
- added C1: 470uF, Capacitor_THT:CP_Radial_D6.3mm_P2.50mm, symbol Device:C_Polarized
- added J1, J3: Conn_01x02_Male, Connector_PinHeader_2.54mm:PinHeader_1x02_P2.54mm_Vertical, symbol Connector:Conn_01x02_Male
- added J14, J2: Conn_01x03_Male, Connector_PinHeader_2.54mm:PinHeader_1x03_P2.54mm_Vertical, symbol Connector:Conn_01x03_Male
- A1: renamed from A?; footprint daisy-seed:Device_Audio_Electrosmith_Daisy_Seed -> Device_Audio_Electrosmith_Daisy_Seed:Device_Audio_Electrosmith_Daisy_Seed
- D2, D3, D4, D5, D6: renamed from D?; footprint (none) -> LED_THT:LED_D5.0mm
- H1, H2, H3, H4: renamed from H?; footprint (none) -> MountingHole:MountingHole_3.2mm_M3
- J4: renamed from J?; footprint (none) -> Connector_PinHeader_2.54mm:PinHeader_1x02_P2.54mm_Vertical
- JP1: renamed from JP?; footprint (none) -> Connector_PinHeader_2.54mm:PinHeader_1x02_P2.54mm_Vertical
- R10, R6, R7, R8, R9: renamed from R?; footprint (none) -> Resistor_SMD:R_0805_2012Metric
- SW1, SW2, SW3, SW4, SW5, SW6, SW7, SW8: renamed from SW?; footprint (none) -> Button_Switch_THT:SW_PUSH_6mm_H4.3mm
- U2, U3: renamed from U?; footprint (none) -> Package_SO:SOIC-16_3.9x9.9mm_P1.27mm
- gave numbers to parts that had none: 7
Connections:
- net GND: now also C1.2, J2.1 (Pin_1)
- net GNDA: now also J1.1 (Pin_1), J3.1 (Pin_1)
- net VCC: now also A1.38 (3V3_D), C1.1
- net midi_in_ring: now reaches R4.2
- net midi_in_ring: now also R1.2, J14.2 (Pin_2), J2.2 (Pin_2)
- net midi_in_tip: now reaches R5.1
- net midi_in_tip: now also D1.2 (A), U1.3 (C2), J14.3 (Pin_3), J2.3 (Pin_3)
- net audio_out_tip: now reaches A1.18 (AUDIO_OUT_L)
- net audio_out_tip: now also J1.2 (Pin_2)
- net audio_in_tip: now reaches A1.16 (AUDIO_IN_L)
- net audio_in_tip: now also J3.2 (Pin_2)
- no-connect marks 28 -> 27
