File: schematics/polymod_proto_1/polymod_proto_1/polymod_proto_1.kicad_sch (KiCad schematic)
At the start: 39 parts, among them J1 Conn_01x02_Male, J14 Conn_01x03_Male, J2 Conn_01x03_Male, J3 Conn_01x02_Male, J4 Barrel_Jack, SW1 SW_Push, SW2 SW_Push, SW3 SW_Push, SW4 SW_Push, SW5 SW_Push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

Commit message: routing started
Parts:
- removed SW6, SW7, SW8: SW_Push, Button_Switch_THT:SW_PUSH-12mm, symbol Switch:SW_Push
Connections:
- no-connect marks 27 -> 33
Changed lines of the file:
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@@
   (no_connect (at 107.95 153.67))
   (no_connect (at 44.45 259.08))
+  (no_connect (at 281.94 140.97))
+  (no_connect (at 295.91 140.97))
+  (no_connect (at 309.88 140.97))
+  (no_connect (at 309.88 130.81))
+  (no_connect (at 295.91 130.81))
+  (no_connect (at 281.94 130.81))
   (wire (pts (xy 76.2 60.96) (xy 80.01 60.96))
     (stroke (width 0) (type default) (color 0 0 0 0))
@@
     (pin "2")
   )
-  (symbol (lib_id "Switch:SW_Push") (at 295.91 135.89 90) (unit 1)
-    (in_bom yes) (on_board yes) (fields_autoplaced)
-    (property "Reference" "SW7" (id 0) (at 297.18 134.6199 90)
-      (effects (font (size 1.27 1.27)) (justify right))
-    )
-    (property "Value" "SW_Push" (id 1) (at 297.18 137.1599 90)
-      (effects (font (size 1.27 1.27)) (justify right))
-    )
-    (property "Footprint" "Button_Switch_THT:SW_PUSH-12mm" (id 2) (at 290.83 135.89 0)
-      (effects (font (size 1.27 1.27)) hide)
-    )
-    (property "Datasheet" "~" (id 3) (at 290.83 135.89 0)
-      (effects (font (size 1.27 1.27)) hide)
-    )
-    (pin "1")
-    (pin "2")
-  )
   (symbol (lib_id "power:GND") (at 356.87 151.13 0) (unit 1)
     (in_bom yes) (on_board yes)
@@
     )
     (property "Datasheet" "~" (id 3) (at 300.99 69.85 0)
-      (effects (font (size 1.27 1.27)) hide)
-    )
-    (pin "1")
-    (pin "2")
-  )
-  (symbol (lib_id "Switch:SW_Push") (at 281.94 135.89 90) (unit 1)
-    (in_bom yes) (on_board yes) (fields_autoplaced)
-    (property "Reference" "SW6" (id 0) (at 283.21 134.6199 90)
-      (effects (font (size 1.27 1.27)) (justify right))
-    )
-    (property "Value" "SW_Push" (id 1) (at 283.21 137.1599 90)
-      (effects (font (size 1.27 1.27)) (justify right))
-    )
-    (property "Footprint" "Button_Switch_THT:SW_PUSH-12mm" (id 2) (at 276.86 135.89 0)
-      (effects (font (size 1.27 1.27)) hide)
-    )
-    (property "Datasheet" "~" (id 3) (at 276.86 135.89 0)
-      (effects (font (size 1.27 1.27)) hide)
-    )
-    (pin "1")
-    (pin "2")
-  )
-  (symbol (lib_id "Switch:SW_Push") (at 309.88 135.89 90) (unit 1)
-    (in_bom yes) (on_board yes) (fields_autoplaced)
-    (property "Reference" "SW8" (id 0) (at 311.15 134.6199 90)
-      (effects (font (size 1.27 1.27)) (justify right))
-    )
-    (property "Value" "SW_Push" (id 1) (at 311.15 137.1599 90)
-      (effects (font (size 1.27 1.27)) (justify right))
-    )
-    (property "Footprint" "Button_Switch_THT:SW_PUSH-12mm" (id 2) (at 304.8 135.89 0)
-      (effects (font (size 1.27 1.27)) hide)
-    )
-    (property "Datasheet" "~" (id 3) (at 304.8 135.89 0)
       (effects (font (size 1.27 1.27)) hide)
     )
@@
       (reference "J4") (unit 1) (value "Barrel_Jack") (footprint "Connector_PinHeader_2.54mm:PinHeader_1x02_P2.54mm_Vertical")
     )
-    (path "/abd8f63e-8fbf-4ad4-a216-38dee4937522/5e6f3146-8d81-4d38-9225-40a455fd4f1f"
-      (reference "J5") (unit 1) (value "AudioJack3") (footprint "")
-    )
     (path "/667335cd-45fc-48b8-8dd3-faf8c21120ea/4e73cd1c-cc94-46f6-8246-5c52d980182a"
       (reference "J6") (unit 1) (value "Conn_01x08_Male") (footprint "Connector_PinSocket_2.54mm:PinSocket_1x08_P2.54mm_Vertical")
@@
       (reference "J14") (unit 1) (value "Conn_01x03_Male") (footprint "Connector_PinHeader_2.54mm:PinHeader_1x03_P2.54mm_Vertical")
     )
-    (path "/0c4f230b-f5e6-413e-a6eb-f32ef4d9b49f/5e6f3146-8d81-4d38-9225-40a455fd4f1f"
-      (reference "J15") (unit 1) (value "AudioJack3") (footprint "")
-    )
     (path "/57fbed25-6dba-42f1-84f1-002a8e5e6d1c"
       (reference "JP1") (unit 1) (value "Jumper_2_Open") (footprint "Connector_PinHeader_2.54mm:PinHeader_1x02_P2.54mm_Vertical")
@@
       (reference "SW5") (unit 1) (value "SW_Push") (footprint "Button_Switch_THT:SW_PUSH-12mm")
     )
-    (path "/61cf1197-d202-4983-a791-bc258c842f49"
-      (reference "SW6") (unit 1) (value "SW_Push") (footprint "Button_Switch_THT:SW_PUSH-12mm")
-    )
-    (path "/2956f6d7-b298-454e-8299-6d4fbebac769"
-      (reference "SW7") (unit 1) (value "SW_Push") (footprint "Button_Switch_THT:SW_PUSH-12mm")
-    )
-    (path "/6348ca7e-00dc-43c7-ade3-29d852ed5791"
-      (reference "SW8") (unit 1) (value "SW_Push") (footprint "Button_Switch_THT:SW_PUSH-12mm")
-    )
     (path "/e9ffe691-9731-424f-ac18-3df8d4dc7459"

Commit message: routing is HARD
Other:
- note added: "removed buttons, no room on PCB!"
Changed lines of the file:
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@@
+    (effects (font (size 1.27 1.27)) (justify left bottom))
+  )
+  (text "removed buttons,\nno room on PCB!" (at 288.29 138.43 0)
     (effects (font (size 1.27 1.27)) (justify left bottom))
   )

Commit message: better layout/routing
Parts:
- removed SW5: SW_Push, Button_Switch_THT:SW_PUSH-12mm, symbol Switch:SW_Push
Connections:
- no-connect marks 33 -> 35
Changed lines of the file:
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@@
   (junction (at 120.65 269.24) (diameter 0) (color 0 0 0 0)
   )
+  (no_connect (at 267.97 140.97))
+  (no_connect (at 267.97 130.81))
   (no_connect (at 369.57 113.03))
   (no_connect (at 344.17 110.49))
@@
     (pin "2")
   )
-  (symbol (lib_id "Switch:SW_Push") (at 267.97 135.89 90) (unit 1)
-    (in_bom yes) (on_board yes) (fields_autoplaced)
-    (property "Reference" "SW5" (id 0) (at 269.24 134.6199 90)
-      (effects (font (size 1.27 1.27)) (justify right))
-    )
-    (property "Value" "SW_Push" (id 1) (at 269.24 137.1599 90)
-      (effects (font (size 1.27 1.27)) (justify right))
-    )
-    (property "Footprint" "Button_Switch_THT:SW_PUSH-12mm" (id 2) (at 262.89 135.89 0)
-      (effects (font (size 1.27 1.27)) hide)
-    )
-    (property "Datasheet" "~" (id 3) (at 262.89 135.89 0)
-      (effects (font (size 1.27 1.27)) hide)
-    )
-    (pin "1")
-    (pin "2")
-  )
   (symbol (lib_id "Device:R") (at 157.48 266.7 270) (unit 1)
     (in_bom yes) (on_board yes)
@@
       (reference "SW4") (unit 1) (value "SW_Push") (footprint "Button_Switch_THT:SW_PUSH-12mm")
     )
-    (path "/ed4fa8e2-d035-4701-85da-5eec53c3cdf1"
-      (reference "SW5") (unit 1) (value "SW_Push") (footprint "Button_Switch_THT:SW_PUSH-12mm")
-    )
     (path "/e9ffe691-9731-424f-ac18-3df8d4dc7459"

Commit message: gerbers!
Parts:
- R1, R10, R2, R3, R4, R5, R6, R7, R8, R9: footprint Resistor_SMD:R_0805_2012Metric -> polymodcustom:R_0805_2012Metric
- SW1, SW2, SW3, SW4: footprint Button_Switch_THT:SW_PUSH-12mm -> polymodcustom:SW_PUSH-12mm
