File: schematics/polymod_proto_1/polymod_proto_1/potgroup.kicad_sch (KiCad schematic)
At the start: 9 parts

Commit message: pcb layout about to start
Parts:
- RV10, RV11, RV12, RV13, RV14, RV15, RV16, RV9: renamed from RV?; footprint (none) -> Potentiometer_THT:Potentiometer_Alps_RK09K_Single_Vertical
- U7: renamed from U?; footprint (none) -> Package_SO:SOIC-16_3.9x9.9mm_P1.27mm
Changed lines of the file:
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@@
   (symbol (lib_id "Device:R_Potentiometer") (at 114.3 137.16 0)
     (in_bom yes) (on_board yes) (fields_autoplaced)
-    (property "Reference" "RV?" (id 0) (at 112.5221 136.2515 0)
+    (property "Reference" "RV14" (id 0) (at 112.5221 136.2515 0)
       (effects (font (size 1.27 1.27)) (justify right))
     )
@@
       (effects (font (size 1.27 1.27)) (justify right))
     )
-    (property "Footprint" "" (id 2) (at 114.3 137.16 0)
+    (property "Footprint" "Potentiometer_THT:Potentiometer_Alps_RK09K_Single_Vertical" (id 2) (at 114.3 137.16 0)
       (effects (font (size 1.27 1.27)) hide)
     )
@@
   (symbol (lib_id "Device:R_Potentiometer") (at 114.3 158.75 0)
     (in_bom yes) (on_board yes) (fields_autoplaced)
-    (property "Reference" "RV?" (id 0) (at 112.5221 157.8415 0)
+    (property "Reference" "RV16" (id 0) (at 112.5221 157.8415 0)
       (effects (font (size 1.27 1.27)) (justify right))
     )
@@
       (effects (font (size 1.27 1.27)) (justify right))
     )
-    (property "Footprint" "" (id 2) (at 114.3 158.75 0)
+    (property "Footprint" "Potentiometer_THT:Potentiometer_Alps_RK09K_Single_Vertical" (id 2) (at 114.3 158.75 0)
       (effects (font (size 1.27 1.27)) hide)
     )
@@
   (symbol (lib_id "Device:R_Potentiometer") (at 114.3 93.98 0)
     (in_bom yes) (on_board yes) (fields_autoplaced)
-    (property "Reference" "RV?" (id 0) (at 112.5221 93.0715 0)
+    (property "Reference" "RV10" (id 0) (at 112.5221 93.0715 0)
       (effects (font (size 1.27 1.27)) (justify right))
     )
@@
       (effects (font (size 1.27 1.27)) (justify right))
     )
-    (property "Footprint" "" (id 2) (at 114.3 93.98 0)
+    (property "Footprint" "Potentiometer_THT:Potentiometer_Alps_RK09K_Single_Vertical" (id 2) (at 114.3 93.98 0)
       (effects (font (size 1.27 1.27)) hide)
     )
@@
   (symbol (lib_id "Device:R_Potentiometer") (at 114.3 105.41 0)
     (in_bom yes) (on_board yes) (fields_autoplaced)
-    (property "Reference" "RV?" (id 0) (at 112.5221 104.5015 0)
+    (property "Reference" "RV11" (id 0) (at 112.5221 104.5015 0)
       (effects (font (size 1.27 1.27)) (justify right))
     )
@@
       (effects (font (size 1.27 1.27)) (justify right))
     )
-    (property "Footprint" "" (id 2) (at 114.3 105.41 0)
+    (property "Footprint" "Potentiometer_THT:Potentiometer_Alps_RK09K_Single_Vertical" (id 2) (at 114.3 105.41 0)
       (effects (font (size 1.27 1.27)) hide)
     )
@@
   (symbol (lib_id "power:GND") (at 87.63 162.56 0)
     (in_bom yes) (on_board yes) (fields_autoplaced)
-    (property "Reference" "#PWR?" (id 0) (at 87.63 168.91 0)
+    (property "Reference" "#PWR018" (id 0) (at 87.63 168.91 0)
       (effects (font (size 1.27 1.27)) hide)
     )
@@
   (symbol (lib_id "power:VCC") (at 130.81 76.2 0)
     (in_bom yes) (on_board yes)
-    (property "Reference" "#PWR?" (id 0) (at 130.81 80.01 0)
+    (property "Reference" "#PWR019" (id 0) (at 130.81 80.01 0)
       (effects (font (size 1.27 1.27)) hide)
     )
@@
   (symbol (lib_id "Device:R_Potentiometer") (at 114.3 127 0)
     (in_bom yes) (on_board yes) (fields_autoplaced)
-    (property "Reference" "RV?" (id 0) (at 112.5221 126.0915 0)
+    (property "Reference" "RV13" (id 0) (at 112.5221 126.0915 0)
       (effects (font (size 1.27 1.27)) (justify right))
     )
@@
       (effects (font (size 1.27 1.27)) (justify right))
     )
-    (property "Footprint" "" (id 2) (at 114.3 127 0)
+    (property "Footprint" "Potentiometer_THT:Potentiometer_Alps_RK09K_Single_Vertical" (id 2) (at 114.3 127 0)
       (effects (font (size 1.27 1.27)) hide)
     )
@@
   (symbol (lib_id "Device:R_Potentiometer") (at 114.3 83.82 0)
     (in_bom yes) (on_board yes) (fields_autoplaced)
-    (property "Reference" "RV?" (id 0) (at 112.5221 82.9115 0)
+    (property "Reference" "RV9" (id 0) (at 112.5221 82.9115 0)
       (effects (font (size 1.27 1.27)) (justify right))
     )
@@
       (effects (font (size 1.27 1.27)) (justify right))
     )
-    (property "Footprint" "" (id 2) (at 114.3 83.82 0)
+    (property "Footprint" "Potentiometer_THT:Potentiometer_Alps_RK09K_Single_Vertical" (id 2) (at 114.3 83.82 0)
       (effects (font (size 1.27 1.27)) hide)
     )
@@
   (symbol (lib_id "Device:R_Potentiometer") (at 114.3 148.59 0)
     (in_bom yes) (on_board yes) (fields_autoplaced)
-    (property "Reference" "RV?" (id 0) (at 112.5221 147.6815 0)
+    (property "Reference" "RV15" (id 0) (at 112.5221 147.6815 0)
       (effects (font (size 1.27 1.27)) (justify right))
     )
@@
       (effects (font (size 1.27 1.27)) (justify right))
     )
-    (property "Footprint" "" (id 2) (at 114.3 148.59 0)
+    (property "Footprint" "Potentiometer_THT:Potentiometer_Alps_RK09K_Single_Vertical" (id 2) (at 114.3 148.59 0)
       (effects (font (size 1.27 1.27)) hide)
     )
@@
   (symbol (lib_id "4xxx:4051") (at 167.64 99.06 0)
     (in_bom yes) (on_board yes)
-    (property "Reference" "U?" (id 0) (at 178.5204 80.0948 0))
+    (property "Reference" "U7" (id 0) (at 178.5204 80.0948 0))
     (property "Value" "4051" (id 1) (at 173.99 74.93 0))
-    (property "Footprint" "" (id 2) (at 167.64 99.06 0)
+    (property "Footprint" "Package_SO:SOIC-16_3.9x9.9mm_P1.27mm" (id 2) (at 167.64 99.06 0)
       (effects (font (size 1.27 1.27)) hide)
     )
@@
   (symbol (lib_id "Device:R_Potentiometer") (at 114.3 115.57 0)
     (in_bom yes) (on_board yes) (fields_autoplaced)
-    (property "Reference" "RV?" (id 0) (at 112.5221 114.6615 0)
+    (property "Reference" "RV12" (id 0) (at 112.5221 114.6615 0)
       (effects (font (size 1.27 1.27)) (justify right))
     )
@@
       (effects (font (size 1.27 1.27)) (justify right))
     )
-    (property "Footprint" "" (id 2) (at 114.3 115.57 0)
+    (property "Footprint" "Potentiometer_THT:Potentiometer_Alps_RK09K_Single_Vertical" (id 2) (at 114.3 115.57 0)
       (effects (font (size 1.27 1.27)) hide)
     )

Commit message: layout going well
Parts:
- renumbered RV9 to RV1, RV10 to RV2, RV11 to RV3, RV12 to RV4, RV13 to RV5, RV14 to RV6, RV15 to RV7, RV16 to RV8, U7 to U4
Changed lines of the file:
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@@
   (symbol (lib_id "Device:R_Potentiometer") (at 114.3 137.16 0)
     (in_bom yes) (on_board yes) (fields_autoplaced)
-    (property "Reference" "RV14" (id 0) (at 112.5221 136.2515 0)
+    (property "Reference" "RV6" (id 0) (at 112.5221 136.2515 0)
       (effects (font (size 1.27 1.27)) (justify right))
     )
@@
   (symbol (lib_id "Device:R_Potentiometer") (at 114.3 158.75 0)
     (in_bom yes) (on_board yes) (fields_autoplaced)
-    (property "Reference" "RV16" (id 0) (at 112.5221 157.8415 0)
+    (property "Reference" "RV8" (id 0) (at 112.5221 157.8415 0)
       (effects (font (size 1.27 1.27)) (justify right))
     )
@@
   (symbol (lib_id "Device:R_Potentiometer") (at 114.3 93.98 0)
     (in_bom yes) (on_board yes) (fields_autoplaced)
-    (property "Reference" "RV10" (id 0) (at 112.5221 93.0715 0)
+    (property "Reference" "RV2" (id 0) (at 112.5221 93.0715 0)
       (effects (font (size 1.27 1.27)) (justify right))
     )
@@
   (symbol (lib_id "Device:R_Potentiometer") (at 114.3 105.41 0)
     (in_bom yes) (on_board yes) (fields_autoplaced)
-    (property "Reference" "RV11" (id 0) (at 112.5221 104.5015 0)
+    (property "Reference" "RV3" (id 0) (at 112.5221 104.5015 0)
       (effects (font (size 1.27 1.27)) (justify right))
     )
@@
   (symbol (lib_id "Device:R_Potentiometer") (at 114.3 127 0)
     (in_bom yes) (on_board yes) (fields_autoplaced)
-    (property "Reference" "RV13" (id 0) (at 112.5221 126.0915 0)
+    (property "Reference" "RV5" (id 0) (at 112.5221 126.0915 0)
       (effects (font (size 1.27 1.27)) (justify right))
     )
@@
   (symbol (lib_id "Device:R_Potentiometer") (at 114.3 83.82 0)
     (in_bom yes) (on_board yes) (fields_autoplaced)
-    (property "Reference" "RV9" (id 0) (at 112.5221 82.9115 0)
+    (property "Reference" "RV1" (id 0) (at 112.5221 82.9115 0)
       (effects (font (size 1.27 1.27)) (justify right))
     )
@@
   (symbol (lib_id "Device:R_Potentiometer") (at 114.3 148.59 0)
     (in_bom yes) (on_board yes) (fields_autoplaced)
-    (property "Reference" "RV15" (id 0) (at 112.5221 147.6815 0)
+    (property "Reference" "RV7" (id 0) (at 112.5221 147.6815 0)
       (effects (font (size 1.27 1.27)) (justify right))
     )
@@
   (symbol (lib_id "4xxx:4051") (at 167.64 99.06 0)
     (in_bom yes) (on_board yes)
-    (property "Reference" "U7" (id 0) (at 178.5204 80.0948 0))
+    (property "Reference" "U4" (id 0) (at 178.5204 80.0948 0))
     (property "Value" "4051" (id 1) (at 173.99 74.93 0))
     (property "Footprint" "Package_SO:SOIC-16_3.9x9.9mm_P1.27mm" (id 2) (at 167.64 99.06 0)
@@
   (symbol (lib_id "Device:R_Potentiometer") (at 114.3 115.57 0)
     (in_bom yes) (on_board yes) (fields_autoplaced)
-    (property "Reference" "RV12" (id 0) (at 112.5221 114.6615 0)
+    (property "Reference" "RV4" (id 0) (at 112.5221 114.6615 0)
       (effects (font (size 1.27 1.27)) (justify right))
     )
