File: schematics/polymod_proto_1/polymod_proto_1/potgroup.kicad_sch (KiCad schematic)
At the start: 10 parts, among them J15 AudioJack3, U7 4051

Commit message: routing started
Parts:
- removed J15: AudioJack3, symbol Connector:AudioJack3
Changed lines of the file:
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@@
     (pin "3")
-  )
-  (symbol (lib_id "Connector:AudioJack3") (at 217.17 90.17 0)
-    (in_bom yes) (on_board yes) (fields_autoplaced)
-    (property "Reference" "J15" (id 0) (at 215.265 82.3935 0))
-    (property "Value" "AudioJack3" (id 1) (at 215.265 85.1686 0))
-    (property "Footprint" "" (id 2) (at 217.17 90.17 0)
-      (effects (font (size 1.27 1.27)) hide)
-    )
-    (property "Datasheet" "~" (id 3) (at 217.17 90.17 0)
-      (effects (font (size 1.27 1.27)) hide)
-    )
-    (pin "R")
-    (pin "S")
-    (pin "T")
   )
   (symbol (lib_id "power:GND") (at 87.63 162.56 0)
