File: schematics/polymod_proto_1/polymod_proto_1/outputgroup.kicad_sch (KiCad schematic)
At the start: 10 parts

Commit message: pcb layout about to start
Parts:
- J10: renamed from J?; footprint (none) -> Connector_PinSocket_2.54mm:PinSocket_1x08_P2.54mm_Vertical
- U10: renamed from U?; footprint (none) -> Package_SO:SOIC-16_3.9x9.9mm_P1.27mm
- gave numbers to parts that had none: 8
Changed lines of the file:
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@@
   (symbol (lib_id "Diode:1N4148") (at 125.73 110.49 180)
     (in_bom yes) (on_board yes)
-    (property "Reference" "D?" (id 0) (at 125.73 105.0036 0))
+    (property "Reference" "D36" (id 0) (at 125.73 105.0036 0))
     (property "Value" "1N4148" (id 1) (at 125.73 107.315 0))
     (property "Footprint" "Diode_THT:D_DO-35_SOD27_P7.62mm_Horizontal" (id 2) (at 125.73 106.045 0)
@@
   (symbol (lib_id "Diode:1N4148") (at 125.73 102.87 180)
     (in_bom yes) (on_board yes)
-    (property "Reference" "D?" (id 0) (at 125.73 97.3836 0))
+    (property "Reference" "D35" (id 0) (at 125.73 97.3836 0))
     (property "Value" "1N4148" (id 1) (at 125.73 99.695 0))
     (property "Footprint" "Diode_THT:D_DO-35_SOD27_P7.62mm_Horizontal" (id 2) (at 125.73 98.425 0)
@@
   (symbol (lib_id "Diode:1N4148") (at 125.73 87.63 180)
     (in_bom yes) (on_board yes)
-    (property "Reference" "D?" (id 0) (at 125.73 82.1436 0))
+    (property "Reference" "D33" (id 0) (at 125.73 82.1436 0))
     (property "Value" "1N4148" (id 1) (at 125.73 84.455 0))
     (property "Footprint" "Diode_THT:D_DO-35_SOD27_P7.62mm_Horizontal" (id 2) (at 125.73 83.185 0)
@@
   (symbol (lib_id "Diode:1N4148") (at 125.73 125.73 180)
     (in_bom yes) (on_board yes)
-    (property "Reference" "D?" (id 0) (at 125.73 120.2436 0))
+    (property "Reference" "D38" (id 0) (at 125.73 120.2436 0))
     (property "Value" "1N4148" (id 1) (at 125.73 122.555 0))
     (property "Footprint" "Diode_THT:D_DO-35_SOD27_P7.62mm_Horizontal" (id 2) (at 125.73 121.285 0)
@@
   (symbol (lib_id "power:GND") (at 91.44 100.33 0)
     (in_bom yes) (on_board yes)
-    (property "Reference" "#PWR?" (id 0) (at 91.44 106.68 0)
+    (property "Reference" "#PWR025" (id 0) (at 91.44 106.68 0)
       (effects (font (size 1.27 1.27)) hide)
     )
@@
   (symbol (lib_id "Connector:Conn_01x08_Male") (at 147.32 78.74 0)
     (in_bom yes) (on_board yes)
-    (property "Reference" "J?" (id 0) (at 150.0632 66.5226 0))
+    (property "Reference" "J10" (id 0) (at 150.0632 66.5226 0))
     (property "Value" "Conn_01x08_Male" (id 1) (at 150.0632 68.834 0))
-    (property "Footprint" "" (id 2) (at 147.32 78.74 0)
+    (property "Footprint" "Connector_PinSocket_2.54mm:PinSocket_1x08_P2.54mm_Vertical" (id 2) (at 147.32 78.74 0)
       (effects (font (size 1.27 1.27)) hide)
     )
@@
   (symbol (lib_id "74xx:74HC595") (at 91.44 82.55 0)
     (in_bom yes) (on_board yes)
-    (property "Reference" "U?" (id 0) (at 85.09 62.23 0))
+    (property "Reference" "U10" (id 0) (at 85.09 62.23 0))
     (property "Value" "74HC595" (id 1) (at 83.82 64.77 0))
-    (property "Footprint" "" (id 2) (at 91.44 82.55 0)
+    (property "Footprint" "Package_SO:SOIC-16_3.9x9.9mm_P1.27mm" (id 2) (at 91.44 82.55 0)
       (effects (font (size 1.27 1.27)) hide)
     )
@@
   (symbol (lib_id "Diode:1N4148") (at 125.73 80.01 180)
     (in_bom yes) (on_board yes)
-    (property "Reference" "D?" (id 0) (at 125.73 74.5236 0))
+    (property "Reference" "D32" (id 0) (at 125.73 74.5236 0))
     (property "Value" "1N4148" (id 1) (at 125.73 76.835 0))
     (property "Footprint" "Diode_THT:D_DO-35_SOD27_P7.62mm_Horizontal" (id 2) (at 125.73 75.565 0)
@@
   (symbol (lib_id "Diode:1N4148") (at 125.73 95.25 180)
     (in_bom yes) (on_board yes)
-    (property "Reference" "D?" (id 0) (at 125.73 89.7636 0))
+    (property "Reference" "D34" (id 0) (at 125.73 89.7636 0))
     (property "Value" "1N4148" (id 1) (at 125.73 92.075 0))
     (property "Footprint" "Diode_THT:D_DO-35_SOD27_P7.62mm_Horizontal" (id 2) (at 125.73 90.805 0)
@@
   (symbol (lib_id "power:VCC") (at 91.44 67.31 0)
     (in_bom yes) (on_board yes)
-    (property "Reference" "#PWR?" (id 0) (at 91.44 71.12 0)
+    (property "Reference" "#PWR024" (id 0) (at 91.44 71.12 0)
       (effects (font (size 1.27 1.27)) hide)
     )
@@
   (symbol (lib_id "Diode:1N4148") (at 125.73 72.39 180)
     (in_bom yes) (on_board yes)
-    (property "Reference" "D?" (id 0) (at 125.73 66.9036 0))
+    (property "Reference" "D31" (id 0) (at 125.73 66.9036 0))
     (property "Value" "1N4148" (id 1) (at 125.73 69.215 0))
     (property "Footprint" "Diode_THT:D_DO-35_SOD27_P7.62mm_Horizontal" (id 2) (at 125.73 67.945 0)
@@
   (symbol (lib_id "Diode:1N4148") (at 125.73 118.11 180)
     (in_bom yes) (on_board yes)
-    (property "Reference" "D?" (id 0) (at 125.73 112.6236 0))
+    (property "Reference" "D37" (id 0) (at 125.73 112.6236 0))
     (property "Value" "1N4148" (id 1) (at 125.73 114.935 0))
     (property "Footprint" "Diode_THT:D_DO-35_SOD27_P7.62mm_Horizontal" (id 2) (at 125.73 113.665 0)

Commit message: layout going well
Parts:
- D10: renamed from D34; footprint Diode_THT:D_DO-35_SOD27_P7.62mm_Horizontal -> Diode_SMD:Nexperia_CFP3_SOD-123W
- D11: renamed from D35; footprint Diode_THT:D_DO-35_SOD27_P7.62mm_Horizontal -> Diode_SMD:Nexperia_CFP3_SOD-123W
- D12: renamed from D36; footprint Diode_THT:D_DO-35_SOD27_P7.62mm_Horizontal -> Diode_SMD:Nexperia_CFP3_SOD-123W
- D13: renamed from D37; footprint Diode_THT:D_DO-35_SOD27_P7.62mm_Horizontal -> Diode_SMD:Nexperia_CFP3_SOD-123W
- D14: renamed from D38; footprint Diode_THT:D_DO-35_SOD27_P7.62mm_Horizontal -> Diode_SMD:Nexperia_CFP3_SOD-123W
- D7: renamed from D31; footprint Diode_THT:D_DO-35_SOD27_P7.62mm_Horizontal -> Diode_SMD:Nexperia_CFP3_SOD-123W
- D8: renamed from D32; footprint Diode_THT:D_DO-35_SOD27_P7.62mm_Horizontal -> Diode_SMD:Nexperia_CFP3_SOD-123W
- D9: renamed from D33; footprint Diode_THT:D_DO-35_SOD27_P7.62mm_Horizontal -> Diode_SMD:Nexperia_CFP3_SOD-123W
- renumbered J10 to J6, U10 to U5
Changed lines of the file:
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@@
   (symbol (lib_id "Diode:1N4148") (at 125.73 110.49 180)
     (in_bom yes) (on_board yes)
-    (property "Reference" "D36" (id 0) (at 125.73 105.0036 0))
+    (property "Reference" "D12" (id 0) (at 125.73 105.0036 0))
     (property "Value" "1N4148" (id 1) (at 125.73 107.315 0))
-    (property "Footprint" "Diode_THT:D_DO-35_SOD27_P7.62mm_Horizontal" (id 2) (at 125.73 106.045 0)
+    (property "Footprint" "Diode_SMD:Nexperia_CFP3_SOD-123W" (id 2) (at 125.73 106.045 0)
       (effects (font (size 1.27 1.27)) hide)
     )
@@
   (symbol (lib_id "Diode:1N4148") (at 125.73 102.87 180)
     (in_bom yes) (on_board yes)
-    (property "Reference" "D35" (id 0) (at 125.73 97.3836 0))
+    (property "Reference" "D11" (id 0) (at 125.73 97.3836 0))
     (property "Value" "1N4148" (id 1) (at 125.73 99.695 0))
-    (property "Footprint" "Diode_THT:D_DO-35_SOD27_P7.62mm_Horizontal" (id 2) (at 125.73 98.425 0)
+    (property "Footprint" "Diode_SMD:Nexperia_CFP3_SOD-123W" (id 2) (at 125.73 98.425 0)
       (effects (font (size 1.27 1.27)) hide)
     )
@@
   (symbol (lib_id "Diode:1N4148") (at 125.73 87.63 180)
     (in_bom yes) (on_board yes)
-    (property "Reference" "D33" (id 0) (at 125.73 82.1436 0))
+    (property "Reference" "D9" (id 0) (at 125.73 82.1436 0))
     (property "Value" "1N4148" (id 1) (at 125.73 84.455 0))
-    (property "Footprint" "Diode_THT:D_DO-35_SOD27_P7.62mm_Horizontal" (id 2) (at 125.73 83.185 0)
+    (property "Footprint" "Diode_SMD:Nexperia_CFP3_SOD-123W" (id 2) (at 125.73 83.185 0)
       (effects (font (size 1.27 1.27)) hide)
     )
@@
   (symbol (lib_id "Diode:1N4148") (at 125.73 125.73 180)
     (in_bom yes) (on_board yes)
-    (property "Reference" "D38" (id 0) (at 125.73 120.2436 0))
+    (property "Reference" "D14" (id 0) (at 125.73 120.2436 0))
     (property "Value" "1N4148" (id 1) (at 125.73 122.555 0))
-    (property "Footprint" "Diode_THT:D_DO-35_SOD27_P7.62mm_Horizontal" (id 2) (at 125.73 121.285 0)
+    (property "Footprint" "Diode_SMD:Nexperia_CFP3_SOD-123W" (id 2) (at 125.73 121.285 0)
       (effects (font (size 1.27 1.27)) hide)
     )
@@
   (symbol (lib_id "power:GND") (at 91.44 100.33 0)
     (in_bom yes) (on_board yes)
-    (property "Reference" "#PWR025" (id 0) (at 91.44 106.68 0)
+    (property "Reference" "#PWR015" (id 0) (at 91.44 106.68 0)
       (effects (font (size 1.27 1.27)) hide)
     )
@@
   (symbol (lib_id "Connector:Conn_01x08_Male") (at 147.32 78.74 0)
     (in_bom yes) (on_board yes)
-    (property "Reference" "J10" (id 0) (at 150.0632 66.5226 0))
+    (property "Reference" "J6" (id 0) (at 150.0632 66.5226 0))
     (property "Value" "Conn_01x08_Male" (id 1) (at 150.0632 68.834 0))
     (property "Footprint" "Connector_PinSocket_2.54mm:PinSocket_1x08_P2.54mm_Vertical" (id 2) (at 147.32 78.74 0)
@@
   (symbol (lib_id "74xx:74HC595") (at 91.44 82.55 0)
     (in_bom yes) (on_board yes)
-    (property "Reference" "U10" (id 0) (at 85.09 62.23 0))
+    (property "Reference" "U5" (id 0) (at 85.09 62.23 0))
     (property "Value" "74HC595" (id 1) (at 83.82 64.77 0))
     (property "Footprint" "Package_SO:SOIC-16_3.9x9.9mm_P1.27mm" (id 2) (at 91.44 82.55 0)
@@
   (symbol (lib_id "Diode:1N4148") (at 125.73 80.01 180)
     (in_bom yes) (on_board yes)
-    (property "Reference" "D32" (id 0) (at 125.73 74.5236 0))
+    (property "Reference" "D8" (id 0) (at 125.73 74.5236 0))
     (property "Value" "1N4148" (id 1) (at 125.73 76.835 0))
-    (property "Footprint" "Diode_THT:D_DO-35_SOD27_P7.62mm_Horizontal" (id 2) (at 125.73 75.565 0)
+    (property "Footprint" "Diode_SMD:Nexperia_CFP3_SOD-123W" (id 2) (at 125.73 75.565 0)
       (effects (font (size 1.27 1.27)) hide)
     )
@@
   (symbol (lib_id "Diode:1N4148") (at 125.73 95.25 180)
     (in_bom yes) (on_board yes)
-    (property "Reference" "D34" (id 0) (at 125.73 89.7636 0))
+    (property "Reference" "D10" (id 0) (at 125.73 89.7636 0))
     (property "Value" "1N4148" (id 1) (at 125.73 92.075 0))
-    (property "Footprint" "Diode_THT:D_DO-35_SOD27_P7.62mm_Horizontal" (id 2) (at 125.73 90.805 0)
+    (property "Footprint" "Diode_SMD:Nexperia_CFP3_SOD-123W" (id 2) (at 125.73 90.805 0)
       (effects (font (size 1.27 1.27)) hide)
     )
@@
   (symbol (lib_id "power:VCC") (at 91.44 67.31 0)
     (in_bom yes) (on_board yes)
-    (property "Reference" "#PWR024" (id 0) (at 91.44 71.12 0)
+    (property "Reference" "#PWR014" (id 0) (at 91.44 71.12 0)
       (effects (font (size 1.27 1.27)) hide)
     )
@@
   (symbol (lib_id "Diode:1N4148") (at 125.73 72.39 180)
     (in_bom yes) (on_board yes)
-    (property "Reference" "D31" (id 0) (at 125.73 66.9036 0))
+    (property "Reference" "D7" (id 0) (at 125.73 66.9036 0))
     (property "Value" "1N4148" (id 1) (at 125.73 69.215 0))
-    (property "Footprint" "Diode_THT:D_DO-35_SOD27_P7.62mm_Horizontal" (id 2) (at 125.73 67.945 0)
+    (property "Footprint" "Diode_SMD:Nexperia_CFP3_SOD-123W" (id 2) (at 125.73 67.945 0)
       (effects (font (size 1.27 1.27)) hide)
     )
@@
   (symbol (lib_id "Diode:1N4148") (at 125.73 118.11 180)
     (in_bom yes) (on_board yes)
-    (property "Reference" "D37" (id 0) (at 125.73 112.6236 0))
+    (property "Reference" "D13" (id 0) (at 125.73 112.6236 0))
     (property "Value" "1N4148" (id 1) (at 125.73 114.935 0))
-    (property "Footprint" "Diode_THT:D_DO-35_SOD27_P7.62mm_Horizontal" (id 2) (at 125.73 113.665 0)
+    (property "Footprint" "Diode_SMD:Nexperia_CFP3_SOD-123W" (id 2) (at 125.73 113.665 0)
       (effects (font (size 1.27 1.27)) hide)
     )

Commit message: components pretty much in place
Parts:
- renumbered D7 to D31, D8 to D32, D9 to D33, D10 to D34, D11 to D35, D12 to D36, D13 to D37, D14 to D38, J6 to J10, U5 to U10
Changed lines of the file:
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@@
   (symbol (lib_id "Diode:1N4148") (at 125.73 110.49 180)
     (in_bom yes) (on_board yes)
-    (property "Reference" "D12" (id 0) (at 125.73 105.0036 0))
+    (property "Reference" "D36" (id 0) (at 125.73 105.0036 0))
     (property "Value" "1N4148" (id 1) (at 125.73 107.315 0))
     (property "Footprint" "Diode_SMD:Nexperia_CFP3_SOD-123W" (id 2) (at 125.73 106.045 0)
@@
   (symbol (lib_id "Diode:1N4148") (at 125.73 102.87 180)
     (in_bom yes) (on_board yes)
-    (property "Reference" "D11" (id 0) (at 125.73 97.3836 0))
+    (property "Reference" "D35" (id 0) (at 125.73 97.3836 0))
     (property "Value" "1N4148" (id 1) (at 125.73 99.695 0))
     (property "Footprint" "Diode_SMD:Nexperia_CFP3_SOD-123W" (id 2) (at 125.73 98.425 0)
@@
   (symbol (lib_id "Diode:1N4148") (at 125.73 87.63 180)
     (in_bom yes) (on_board yes)
-    (property "Reference" "D9" (id 0) (at 125.73 82.1436 0))
+    (property "Reference" "D33" (id 0) (at 125.73 82.1436 0))
     (property "Value" "1N4148" (id 1) (at 125.73 84.455 0))
     (property "Footprint" "Diode_SMD:Nexperia_CFP3_SOD-123W" (id 2) (at 125.73 83.185 0)
@@
   (symbol (lib_id "Diode:1N4148") (at 125.73 125.73 180)
     (in_bom yes) (on_board yes)
-    (property "Reference" "D14" (id 0) (at 125.73 120.2436 0))
+    (property "Reference" "D38" (id 0) (at 125.73 120.2436 0))
     (property "Value" "1N4148" (id 1) (at 125.73 122.555 0))
     (property "Footprint" "Diode_SMD:Nexperia_CFP3_SOD-123W" (id 2) (at 125.73 121.285 0)
@@
   (symbol (lib_id "power:GND") (at 91.44 100.33 0)
     (in_bom yes) (on_board yes)
-    (property "Reference" "#PWR015" (id 0) (at 91.44 106.68 0)
+    (property "Reference" "#PWR025" (id 0) (at 91.44 106.68 0)
       (effects (font (size 1.27 1.27)) hide)
     )
@@
   (symbol (lib_id "Connector:Conn_01x08_Male") (at 147.32 78.74 0)
     (in_bom yes) (on_board yes)
-    (property "Reference" "J6" (id 0) (at 150.0632 66.5226 0))
+    (property "Reference" "J10" (id 0) (at 150.0632 66.5226 0))
     (property "Value" "Conn_01x08_Male" (id 1) (at 150.0632 68.834 0))
     (property "Footprint" "Connector_PinSocket_2.54mm:PinSocket_1x08_P2.54mm_Vertical" (id 2) (at 147.32 78.74 0)
@@
   (symbol (lib_id "74xx:74HC595") (at 91.44 82.55 0)
     (in_bom yes) (on_board yes)
-    (property "Reference" "U5" (id 0) (at 85.09 62.23 0))
+    (property "Reference" "U10" (id 0) (at 85.09 62.23 0))
     (property "Value" "74HC595" (id 1) (at 83.82 64.77 0))
     (property "Footprint" "Package_SO:SOIC-16_3.9x9.9mm_P1.27mm" (id 2) (at 91.44 82.55 0)
@@
   (symbol (lib_id "Diode:1N4148") (at 125.73 80.01 180)
     (in_bom yes) (on_board yes)
-    (property "Reference" "D8" (id 0) (at 125.73 74.5236 0))
+    (property "Reference" "D32" (id 0) (at 125.73 74.5236 0))
     (property "Value" "1N4148" (id 1) (at 125.73 76.835 0))
     (property "Footprint" "Diode_SMD:Nexperia_CFP3_SOD-123W" (id 2) (at 125.73 75.565 0)
@@
   (symbol (lib_id "Diode:1N4148") (at 125.73 95.25 180)
     (in_bom yes) (on_board yes)
-    (property "Reference" "D10" (id 0) (at 125.73 89.7636 0))
+    (property "Reference" "D34" (id 0) (at 125.73 89.7636 0))
     (property "Value" "1N4148" (id 1) (at 125.73 92.075 0))
     (property "Footprint" "Diode_SMD:Nexperia_CFP3_SOD-123W" (id 2) (at 125.73 90.805 0)
@@
   (symbol (lib_id "power:VCC") (at 91.44 67.31 0)
     (in_bom yes) (on_board yes)
-    (property "Reference" "#PWR014" (id 0) (at 91.44 71.12 0)
+    (property "Reference" "#PWR024" (id 0) (at 91.44 71.12 0)
       (effects (font (size 1.27 1.27)) hide)
     )
@@
   (symbol (lib_id "Diode:1N4148") (at 125.73 72.39 180)
     (in_bom yes) (on_board yes)
-    (property "Reference" "D7" (id 0) (at 125.73 66.9036 0))
+    (property "Reference" "D31" (id 0) (at 125.73 66.9036 0))
     (property "Value" "1N4148" (id 1) (at 125.73 69.215 0))
     (property "Footprint" "Diode_SMD:Nexperia_CFP3_SOD-123W" (id 2) (at 125.73 67.945 0)
@@
   (symbol (lib_id "Diode:1N4148") (at 125.73 118.11 180)
     (in_bom yes) (on_board yes)
-    (property "Reference" "D13" (id 0) (at 125.73 112.6236 0))
+    (property "Reference" "D37" (id 0) (at 125.73 112.6236 0))
     (property "Value" "1N4148" (id 1) (at 125.73 114.935 0))
     (property "Footprint" "Diode_SMD:Nexperia_CFP3_SOD-123W" (id 2) (at 125.73 113.665 0)
